File: Teensy_24V_INPUT_OUTPUT.kicad_sch (KiCad schematic)
At the start: 144 parts, among them J1 Conn_01x24, J11 Conn_01x10, J12 Conn_01x10, J13 Conn_01x10, J14 Conn_01x06, J2 Conn_01x24, J3 Screw_Terminal_01x05, J4 Screw_Terminal_01x05, J5 Screw_Terminal_01x05, J6 Screw_Terminal_01x05, J7 Screw_Terminal_01x04, J8 Screw_Terminal_01x04, J9 Screw_Terminal_01x02, Q1 AO3406, Q10 AO3406, Q11 AO3406, Q12 AO3406, Q13 AO3406, Q14 AO3406, Q2 AO3406, Q3 AO3406, Q4 AO3406, Q5 AO3406, Q6 AO3406, Q7 AO3406, Q8 AO3406, Q9 AO3406, U1 LTV-814S-TA1, U10 LTV-814S-TA1, U11 LTV-814S-TA1, U12 LTV-814S-TA1, U13 LTV-814S-TA1, U14 LTV-814S-TA1, U15 LTV-814S-TA1, U16 LTV-814S-TA1, U17 LTV-814S-TA1, U18 LTV-814S-TA1, U19 LTV-814S-TA1, U2 LTV-814S-TA1, U20 LTV-814S-TA1, U21 LM5007MM, U22 CX240D5, U23 CX240D5, U24 CX240D5, U25 CX240D5, U26 CX240D5, U27 CX240D5, U28 CX240D5, U29 CX240D5, U3 LTV-814S-TA1, U30 CX240D5, U31 CX240D5, U32 CX240D5, U33 CX240D5, U34 CX240D5, U35 CX240D5, U4 LTV-814S-TA1, U5 LTV-814S-TA1, U6 LTV-814S-TA1, U7 LTV-814S-TA1, U8 LTV-814S-TA1, U9 LTV-814S-TA1

Commit message: controls only dc now wiht mosfet. limited 30V
Parts:
- removed R46, R59, R60, R61, R66, R67, R68, R69, R72, R73: 1k, symbol Device:R_Small_US
- removed R62, R63, R64, R65: 100, symbol Device:R_Small_US
- removed U22, U23, U24, U25, U26, U27, U28, U29, U30, U31, U32, U33, U34, U35: CX240D5, Package_SIP:SIP4_Sharp-SSR_P7.62mm_Straight, symbol Relay_SolidState:S116S02
- R49, R51, R53, R58: value 1k -> 100; LCSC C106235 -> C11702
Connections:
- net P0 is gone; now on net Output_1: J1.2 (Pin_2)
- net P1 is gone; now on net Output_2: J1.3 (Pin_3)
- net P10 is gone; now on net Output_11: J1.12 (Pin_12)
- net P11 is gone; now on net Output_12: J1.13 (Pin_13)
- net P12 is gone; now on net Output_13: J1.14 (Pin_14)
- net P13 is gone; now on net Input_11: J2.14 (Pin_14)
- net P14 is gone; now on net Input_10: J2.13 (Pin_13)
- net P15 is gone; now on net Input_9: J2.12 (Pin_12)
- net P16 is gone; now on net Input_8: J2.11 (Pin_11)
- net P17 is gone; now on net Input_7: J2.10 (Pin_10)
- net P18 is gone; now on net Input_6: J2.9 (Pin_9)
- net P19 is gone; now on net Input_5: J2.8 (Pin_8)
- net P2 is gone; now on net Output_3: J1.4 (Pin_4)
- net P20 is gone; now on net Input_4: J2.7 (Pin_7)
- net P21 is gone; now on net Input_3: J2.6 (Pin_6)
- net P22 is gone; now on net Input_2: J2.5 (Pin_5)
- net P23 is gone; now on net Input_1: J2.4 (Pin_4)
- net P24 is gone; now on net Output_14: J1.16 (Pin_16)
- net P3 is gone; now on net Output_4: J1.5 (Pin_5)
- net P34 is gone; now on net Input_19: J2.23 (Pin_23)
- net P35 is gone; now on net Input_18: J2.22 (Pin_22)
- net P36 is gone; now on net Input_17: J2.21 (Pin_21)
- net P37 is gone; now on net Input_16: J2.20 (Pin_20)
- net P38 is gone; now on net Input_15: J2.19 (Pin_19)
- net P39 is gone; now on net Input_14: J2.18 (Pin_18)
- net P4 is gone; now on net Output_5: J1.6 (Pin_6)
- net P40 is gone; now on net Input_13: J2.17 (Pin_17)
- net P41 is gone; now on net Input_12: J2.16 (Pin_16)
- net P5 is gone; now on net Output_6: J1.7 (Pin_7)
- net P6 is gone; now on net Output_7: J1.8 (Pin_8)
- net P7 is gone; now on net Output_8: J1.9 (Pin_9)
- net P8 is gone; now on net Output_9: J1.10 (Pin_10)
- net P9 is gone; now on net Output_10: J1.11 (Pin_11)
- net PS1 is gone; now on net GND: J11.1 (Pin_1)
- net +5V: no longer R49.1, R51.1, R53.1, R58.1
- net GND: now also J12.1 (Pin_1), J13.1 (Pin_1), J14.1 (Pin_1)
- net Input_2: no longer R6.2, U3.4
- net Output_1: now also R54.1, R58.1
- net Output_2: now also R49.1, R55.1
- net Output_3: now also R51.1, R56.1
- net Output_4: now also R53.1, R57.1
- net Output_5: no longer R57.1
- net Output_6: no longer R54.1
- net Output_7: no longer R55.1
- net Output_8: no longer R56.1
- net at R56.2: now also Q10.1 (G); no longer Q7.1 (G)
- net at Q7.3 (D): now also J12.9 (Pin_9)
- net at R54.2: now also Q8.1 (G); no longer Q5.1 (G)
- net at Q5.3 (D): now also J12.5 (Pin_5)
- net at J12.3 (Pin_3): now also Q8.3 (D)
- net at J12.7 (Pin_7): now also Q6.3 (D)
- net at J14.5 (Pin_5): now also Q14.3 (D)
- net at Q1.3 (D): now also J11.3 (Pin_3)
- net at R51.2: now also Q6.1 (G)
- net at J11.5 (Pin_5): now also Q2.3 (D)
- net at R49.2: now also Q5.1 (G)
- net at R57.2: now also Q11.1 (G); no longer Q8.1 (G)
- net at J13.3 (Pin_3): now also Q12.3 (D)
- net at J13.5 (Pin_5): now also Q9.3 (D)
- net at J13.7 (Pin_7): now also Q10.3 (D)
- net at J13.9 (Pin_9): now also Q11.3 (D)
- net at R58.2: now also Q12.1 (G)
- net at J14.3 (Pin_3): now also Q13.3 (D)
- net at J11.7 (Pin_7): now also Q3.3 (D)
- net at Q9.1 (G): now also R55.2
- net at J11.9 (Pin_9): now also Q4.3 (D)
- net at R53.2: now also Q7.1 (G)
- net P33 renamed Input_20
- net Input_20: now also R6.2, U3.4
- net PS2: no longer names the net of J11.10 (Pin_10), J11.2 (Pin_2), J11.4 (Pin_4), J11.6 (Pin_6), J11.8 (Pin_8)
- net PS2: no longer J12.1 (Pin_1)
- net PS3: no longer names the net of J12.10 (Pin_10), J12.2 (Pin_2), J12.4 (Pin_4), J12.6 (Pin_6), J12.8 (Pin_8)
- net PS3: no longer J13.1 (Pin_1)
- net PS4: no longer names the net of J13.10 (Pin_10), J13.2 (Pin_2), J13.4 (Pin_4), J13.6 (Pin_6), J13.8 (Pin_8)
